Commit message: 1. Ubuntu 22.04 ROS humble. 2. PCL segmentation. 3. scene segmentation with fastseg

File: simulation/webots_ros2_suv/resource/suv.urdf (robot description, URDF)
Before this commit: robot SUV, 27 links, 28 joints
Links:
- added link range_finder
Joints:
- added joint base_link_range_finder_joint: type fixed, parent base_link, child range_finder, origin xyz=1.73 0 1.38 rpy=-1.570796 0 -1.570796

Commit message: left camera added

File: simulation/webots_ros2_suv/resource/suv.urdf (robot description, URDF)
Before this commit: robot SUV, 28 links, 29 joints
Links:
- added link left_wing_camera
Joints:
- added joint base_link_camera_left_joint: type fixed, parent base_link, child left_wing_camera, origin xyz=1.73 0 1.38 rpy=-1.570796 0 -1.570796
